File: PCB-KiCad/HMS_8ValveDriver.kicad_pcb (KiCad board)
At the start: 2 copper layers, 101.6 x 50.8 mm, 24 parts, among them IC1 ULQ2803A, J1 CONN_10", J10 Valve 3, J11 Valve 2, J12 Valve 1, J15 BNCPTH, J16 BNCPTH, J17 BNCPTH, J18 BNCPTH, J4 POWER_JACK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

Commit message: Update BOM; Generate Gerbers
Other:
- board text added: "Gnd"
- board text added: "V1"
- board text added: "V2"
- board text added: "V3"
- board text added: "V4"
- board text added: "V5"
- board text added: "V6"
- board text added: "V7"
- board text added: "V8"
- board text added: "v1.3 • Sept 2023 • OM"
- board text removed: "Gnd V1 V2 V3 V4 V5 V6 V7 V8 Gnd"
- board text removed: "v1.2.1 • Aug 2023 • OM"
