File: PCB-KiCad/HMS_8ValveDriver.kicad_sch (KiCad schematic)
At the start: 23 parts, among them IC1 ULQ2803A, J1 CONN_10{dblquote}, J10 Valve 3, J11 Valve 2, J12 Valve 1, J15 BNCPTH, J16 BNCPTH, J17 BNCPTH, J18 BNCPTH, J4 POWER_JACK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

Commit message: Update BOM; Generate Gerbers
Other:
- company: (none) -> HMS Research Instrumentation Core
- title: (none) -> 8-Channel Valve Driver
- moved on the sheet: S1, S2, S3, S4
Changed lines of the file:
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@@
 (kicad_sch (version 20230121) (generator eeschema)
   (paper "USLetter")
-  (junction (at 154.94 127) (diameter 0) (color 0 0 0 0)
-  )
-  (junction (at 154.94 119.38) (diameter 0) (color 0 0 0 0)
-  )
-  (junction (at 154.94 134.62) (diameter 0) (color 0 0 0 0)
+  (title_block
+    (title "8-Channel Valve Driver")
+    (date "2023-09-22")
+    (rev "1.3")
+    (company "HMS Research Instrumentation Core")
+  )
+  (junction (at 138.43 116.84) (diameter 0) (color 0 0 0 0)
+  )
+  (junction (at 138.43 109.22) (diameter 0) (color 0 0 0 0)
+  )
+  (junction (at 138.43 124.46) (diameter 0) (color 0 0 0 0)
   )
   (junction (at 167.64 40.64) (diameter 0) (color 0 0 0 0)
@@
     (stroke (width 0.1524) (type solid))
   )
-  (wire (pts (xy 154.94 127) (xy 154.94 119.38))
+  (wire (pts (xy 138.43 116.84) (xy 138.43 109.22))
     (stroke (width 0.1524) (type solid))
   )
@@
     (stroke (width 0.1524) (type solid))
   )
-  (wire (pts (xy 144.78 111.76) (xy 137.16 111.76))
+  (wire (pts (xy 128.27 101.6) (xy 120.65 101.6))
     (stroke (width 0.1524) (type solid))
   )
@@
     (stroke (width 0.1524) (type solid))
   )
-  (wire (pts (xy 154.94 172.72) (xy 154.94 134.62))
+  (wire (pts (xy 138.43 162.56) (xy 138.43 124.46))
     (stroke (width 0.1524) (type solid))
   )
@@
     (stroke (width 0.1524) (type solid))
   )
-  (wire (pts (xy 154.94 119.38) (xy 154.94 111.76))
+  (wire (pts (xy 138.43 109.22) (xy 138.43 101.6))
     (stroke (width 0.1524) (type solid))
   )
@@
     (stroke (width 0.1524) (type solid))
   )
-  (wire (pts (xy 154.94 134.62) (xy 154.94 127))
+  (wire (pts (xy 138.43 124.46) (xy 138.43 116.84))
     (stroke (width 0.1524) (type solid))
   )
@@
     (stroke (width 0.1524) (type solid))
   )
-  (wire (pts (xy 144.78 119.38) (xy 137.16 119.38))
+  (wire (pts (xy 128.27 109.22) (xy 120.65 109.22))
     (stroke (width 0.1524) (type solid))
   )
@@
     (stroke (width 0.1524) (type solid))
   )
-  (wire (pts (xy 144.78 127) (xy 137.16 127))
+  (wire (pts (xy 128.27 116.84) (xy 120.65 116.84))
     (stroke (width 0.1524) (type solid))
   )
@@
     (stroke (width 0.1524) (type solid))
   )
-  (wire (pts (xy 144.78 134.62) (xy 137.16 134.62))
+  (wire (pts (xy 128.27 124.46) (xy 120.65 124.46))
     (stroke (width 0.1524) (type solid))
   )
@@
     (effects (font (size 0.889 0.889)) (justify left bottom))
   )
-  (label "V2OUT" (at 137.16 119.38 180) (fields_autoplaced)
+  (label "V2OUT" (at 120.65 109.22 180) (fields_autoplaced)
     (effects (font (size 0.889 0.889)) (justify right bottom))
   )
@@
     (effects (font (size 0.889 0.889)) (justify left bottom))
   )
-  (label "V4OUT" (at 137.16 134.62 180) (fields_autoplaced)
+  (label "V4OUT" (at 120.65 124.46 180) (fields_autoplaced)
     (effects (font (size 0.889 0.889)) (justify right bottom))
   )
@@
     (effects (font (size 0.889 0.889)) (justify left bottom))
   )
-  (label "V1OUT" (at 137.16 111.76 180) (fields_autoplaced)
+  (label "V1OUT" (at 120.65 101.6 180) (fields_autoplaced)
     (effects (font (size 0.889 0.889)) (justify right bottom))
   )
@@
     (effects (font (size 0.889 0.889)) (justify left bottom))
   )
-  (label "V3OUT" (at 137.16 127 180) (fields_autoplaced)
+  (label "V3OUT" (at 120.65 116.84 180) (fields_autoplaced)
     (effects (font (size 0.889 0.889)) (justify right bottom))
   )
@@
     )
   )
-  (symbol (lib_id "HMS_8ValveDriver-eagle-import:MOMENTARY-SWITCH-SPST-PTH-6.0MM") (at 149.86 134.62 0) (unit 1)
-    (in_bom yes) (on_board yes) (dnp no)
-    (property "Reference" "S4" (at 149.86 133.096 0)
+  (symbol (lib_id "HMS_8ValveDriver-eagle-import:MOMENTARY-SWITCH-SPST-PTH-6.0MM") (at 133.35 124.46 0) (unit 1)
+    (in_bom yes) (on_board yes) (dnp no)
+    (property "Reference" "S4" (at 133.35 122.936 0)
       (effects (font (size 1.778 1.778)) (justify bottom))
     )
-    (property "Value" "MOMENTARY-SWITCH-SPST-PTH-6.0MM" (at 149.86 135.128 0)
+    (property "Value" "MOMENTARY-SWITCH-SPST-PTH-6.0MM" (at 133.35 124.968 0)
       (effects (font (size 1.778 1.778)) (justify top))
     )
-    (property "Footprint" "HMS_8ValveDriver:TACTILE_SWITCH_PTH_6.0MM" (at 149.86 134.62 0)
-      (effects (font (size 1.27 1.27)) hide)
-    )
-    (property "Datasheet" "" (at 149.86 134.62 0)
+    (property "Footprint" "HMS_8ValveDriver:TACTILE_SWITCH_PTH_6.0MM" (at 133.35 124.46 0)
+      (effects (font (size 1.27 1.27)) hide)
+    )
+    (property "Datasheet" "" (at 133.35 124.46 0)
       (effects (font (size 1.27 1.27)) hide)
     )
@@
     )
   )
-  (symbol (lib_id "HMS_8ValveDriver-eagle-import:MOMENTARY-SWITCH-SPST-PTH-6.0MM") (at 149.86 119.38 0) (unit 1)
-    (in_bom yes) (on_board yes) (dnp no)
-    (property "Reference" "S2" (at 149.86 117.856 0)
+  (symbol (lib_id "HMS_8ValveDriver-eagle-import:MOMENTARY-SWITCH-SPST-PTH-6.0MM") (at 133.35 109.22 0) (unit 1)
+    (in_bom yes) (on_board yes) (dnp no)
+    (property "Reference" "S2" (at 133.35 107.696 0)
       (effects (font (size 1.778 1.778)) (justify bottom))
     )
-    (property "Value" "MOMENTARY-SWITCH-SPST-PTH-6.0MM" (at 149.86 119.888 0)
+    (property "Value" "MOMENTARY-SWITCH-SPST-PTH-6.0MM" (at 133.35 109.728 0)
       (effects (font (size 1.778 1.778)) (justify top))
     )
-    (property "Footprint" "HMS_8ValveDriver:TACTILE_SWITCH_PTH_6.0MM" (at 149.86 119.38 0)
-      (effects (font (size 1.27 1.27)) hide)
-    )
-    (property "Datasheet" "" (at 149.86 119.38 0)
+    (property "Footprint" "HMS_8ValveDriver:TACTILE_SWITCH_PTH_6.0MM" (at 133.35 109.22 0)
+      (effects (font (size 1.27 1.27)) hide)
+    )
+    (property "Datasheet" "" (at 133.35 109.22 0)
       (effects (font (size 1.27 1.27)) hide)
     )
@@
     )
   )
-  (symbol (lib_id "HMS_8ValveDriver-eagle-import:MOMENTARY-SWITCH-SPST-PTH-6.0MM") (at 149.86 111.76 0) (unit 1)
-    (in_bom yes) (on_board yes) (dnp no)
-    (property "Reference" "S1" (at 149.86 110.236 0)
+  (symbol (lib_id "HMS_8ValveDriver-eagle-import:MOMENTARY-SWITCH-SPST-PTH-6.0MM") (at 133.35 101.6 0) (unit 1)
+    (in_bom yes) (on_board yes) (dnp no)
+    (property "Reference" "S1" (at 133.35 100.076 0)
       (effects (font (size 1.778 1.778)) (justify bottom))
     )
-    (property "Value" "MOMENTARY-SWITCH-SPST-PTH-6.0MM" (at 149.86 112.268 0)
+    (property "Value" "MOMENTARY-SWITCH-SPST-PTH-6.0MM" (at 133.35 102.108 0)
       (effects (font (size 1.778 1.778)) (justify top))
     )
-    (property "Footprint" "HMS_8ValveDriver:TACTILE_SWITCH_PTH_6.0MM" (at 149.86 111.76 0)
-      (effects (font (size 1.27 1.27)) hide)
-    )
-    (property "Datasheet" "" (at 149.86 111.76 0)
+    (property "Footprint" "HMS_8ValveDriver:TACTILE_SWITCH_PTH_6.0MM" (at 133.35 101.6 0)
+      (effects (font (size 1.27 1.27)) hide)
+    )
+    (property "Datasheet" "" (at 133.35 101.6 0)
       (effects (font (size 1.27 1.27)) hide)
     )
@@
     )
   )
-  (symbol (lib_id "HMS_8ValveDriver-eagle-import:MOMENTARY-SWITCH-SPST-PTH-6.0MM") (at 149.86 127 0) (unit 1)
-    (in_bom yes) (on_board yes) (dnp no)
-    (property "Reference" "S3" (at 149.86 125.476 0)
+  (symbol (lib_id "HMS_8ValveDriver-eagle-import:MOMENTARY-SWITCH-SPST-PTH-6.0MM") (at 133.35 116.84 0) (unit 1)
+    (in_bom yes) (on_board yes) (dnp no)
+    (property "Reference" "S3" (at 133.35 115.316 0)
       (effects (font (size 1.778 1.778)) (justify bottom))
     )
-    (property "Value" "MOMENTARY-SWITCH-SPST-PTH-6.0MM" (at 149.86 127.508 0)
+    (property "Value" "MOMENTARY-SWITCH-SPST-PTH-6.0MM" (at 133.35 117.348 0)
       (effects (font (size 1.778 1.778)) (justify top))
     )
-    (property "Footprint" "HMS_8ValveDriver:TACTILE_SWITCH_PTH_6.0MM" (at 149.86 127 0)
-      (effects (font (size 1.27 1.27)) hide)
-    )
-    (property "Datasheet" "" (at 149.86 127 0)
+    (property "Footprint" "HMS_8ValveDriver:TACTILE_SWITCH_PTH_6.0MM" (at 133.35 116.84 0)
+      (effects (font (size 1.27 1.27)) hide)
+    )
+    (property "Datasheet" "" (at 133.35 116.84 0)
       (effects (font (size 1.27 1.27)) hide)
     )
@@
     )
   )
-  (symbol (lib_id "HMS_8ValveDriver-eagle-import:GND") (at 154.94 175.26 0) (unit 1)
-    (in_bom yes) (on_board yes) (dnp no)
-    (property "Reference" "#GND01" (at 154.94 175.26 0)
-      (effects (font (size 1.27 1.27)) hide)
-    )
-    (property "Value" "GND" (at 154.94 175.514 0)
+  (symbol (lib_id "HMS_8ValveDriver-eagle-import:GND") (at 138.43 165.1 0) (unit 1)
+    (in_bom yes) (on_board yes) (dnp no)
+    (property "Reference" "#GND01" (at 138.43 165.1 0)
+      (effects (font (size 1.27 1.27)) hide)
+    )
+    (property "Value" "GND" (at 138.43 165.354 0)
       (effects (font (size 1.778 1.5113)) (justify top))
     )
-    (property "Footprint" "" (at 154.94 175.26 0)
-      (effects (font (size 1.27 1.27)) hide)
-    )
-    (property "Datasheet" "" (at 154.94 175.26 0)
-      (effects (font (size 1.27 1.27)) hide)
-    )
+    (property "Footprint" "" (at 138.43 165.1 0)
+      (effects (font (size 1.27 1.27)) hide)
+    )
+    (property "Datasheet" "" (at 138.43 165.1 0)
+      (effects (font (size 1.27 1.27)) hide)
+    )
